File: AutoSteerPCB/diyAutoSteer.brd (EAGLE design)
At the start: 127 x 99.1 mm, 65 parts, among them IC2 7805, IC3 7805, J1 I2C Out, J6 Reset, K4 CB1-P-12V, M1 ARDUINO-NANO-3.0, U2 ADC-4CH-ADS1115

Commit message: Added ADS1115 to parts
Missed part, change R8 to zero ohms
Parts:
- R8: value 47 -> 0
Changed lines of the file:
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@@
 <attribute name="VALUE" x="11.557" y="43.18" size="0.6096" layer="27" font="vector" ratio="20" rot="R90"/>
 </element>
-<element name="R8" library="rcl" package="0309/12" value="47" x="41.91" y="62.23" smashed="yes" rot="R180">
+<element name="R8" library="rcl" package="0309/12" value="0" x="41.91" y="62.23" smashed="yes" rot="R180">
 <attribute name="NAME" x="46.101" y="60.325" size="1.27" layer="25" ratio="10" rot="R180"/>
 <attribute name="VALUE" x="45.085" y="62.9158" size="1.27" layer="27" ratio="10" rot="R180"/>

Commit message: v2 PCB
v2 PCB
Parts:
- removed 12S5: WIREPAD3,81/1,1, wirepad:3,81/1,1
- removed A1: A2, SparkFun-Connectors:1X02_LONGPADS
- removed D5, INT0: (no value), SparkFun-Connectors:1X01_LONGPAD
- added +5V_OUT, ANALOGIN: (no value), SparkFun-Connectors:1X03_LONGPADS
- added J2: Pins, SparkFun-Connectors:1X02_LONGPADS
- D2: value 1N4004 -> 3A diode; device diode:DO41-10 -> diode:DO27-15
- moved REMOTE 127.0 mm to (135.9, 8.89), turned to 180 degrees
- moved OK3 117.3 mm to (135.9, 21.6), turned to 270 degrees
- moved R3 111.7 mm to (135.9, 27.9), turned to 0 degrees
- moved IMP 111.1 mm to (118.1, 8.89), turned to 180 degrees
- moved R5 107.6 mm to (135.9, 33.0), turned to 180 degrees
- moved R4 101.9 mm to (127.0, 27.9), turned to 90 degrees
- moved OK1 100.5 mm to (119.4, 21.6), turned to 270 degrees
- moved STEER 99.3 mm to (101.6, 8.89), turned to 180 degrees
- moved D3 98.8 mm to (85.1, 12.7), turned to 90 degrees
- moved GN5 95.5 mm to (12.7, 20.3), turned to 180 degrees
- moved GN4 94.4 mm to (12.7, 10.2)
- moved GN1 93.3 mm to (12.7, 15.2)
- moved R13 92.7 mm to (118.1, 27.9), turned to 180 degrees
- moved GN3 92.6 mm to (27.9, 10.2), turned to 0 degrees
- moved BAT1 90.3 mm to (50.8, 8.89), turned to 180 degrees
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Connections:
- removed net N$9: D5.1, M1.J1.8
- new net N$14: ANALOGIN.2, M1.J2.11
- new net N$18: J2.1, M1.J1.8
- net +5V: now also +5V_OUT.1, +5V_OUT.2, +5V_OUT.3
- net BATT: now also K4.86; no longer K4.85
- net N$10: now also ANALOGIN.3, M1.J2.12; no longer A1.1, M1.J2.10
- net N$15: now also ANALOGIN.1, M1.J2.10; no longer A1.2, M1.J2.11
- net N$24: now also K4.85; no longer K4.86
- net N$6: now also J2.2; no longer INT0.1
- net SW_RAW: no longer 12S5.1
Routing:
- net N$6: track 7.67 -> 41.3 mm
- net N$18: track 0.00 -> 33.3 mm
- net N$11: track 58.3 -> 89.5 mm
- net SCL: track 46.4 -> 15.5 mm, vias 1 -> 0
- net SDA: track 49.2 -> 19.4 mm
- net N$8: track 6.35 -> 34.9 mm
- net N$5: track 44.6 -> 71.9 mm
- net N$14: track 0.00 -> 25.2 mm
- net SW_RAW: track 0.00 -> 24.2 mm, vias 5 -> 4
- net N$21: track 8.15 -> 31.7 mm
- net N$4: track 43.1 -> 66.1 mm
- net N$17: track 17.9 -> 40.6 mm
- net N$19: track 13.5 -> 31.7 mm
- net N$2: track 10.7 -> 28.2 mm
- net N$1: track 13.6 -> 29.2 mm
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Other:
- board size 127 x 99.1 mm -> 148.6 x 100.3 mm
- board text added: "+12 O C"
- board text added: "+12v Battery In"
- board text added: "A0"
- board text added: "D2"
- board text added: "D5"
- board text removed: "+15"
- board text removed: "Batt"
- board text removed: "Gnd O"

Commit message: Version 2
Version 2 of PCB
Parts:
- added +12V, DOG2: (no value), SparkFun-Connectors:1X02_LONGPADS
- moved C21 4.02 mm to (50.8, 59.7)
- moved +5V_OUT 3.81 mm to (52.1, 77.5)
- moved STEER 2.84 mm to (102.9, 11.4)
- moved GN1 2.54 mm to (15.2, 15.2), turned to 90 degrees
- moved GN4 2.54 mm to (15.2, 10.2)
- moved GN5 2.54 mm to (15.2, 20.3)
- moved GN2 2.54 mm to (30.5, 15.2)
- moved GN3 2.54 mm to (30.5, 10.2)
- moved GND 2.54 mm to (30.5, 20.3)
- moved IMP 2.54 mm to (118.1, 11.4)
- moved REMOTE 2.54 mm to (135.9, 11.4)
- moved ON_OFF 1.27 mm to (85.1, 27.9)
- moved D2 1.27 mm to (64.8, 45.7)
- moved R5 1.27 mm to (135.9, 31.8)
Connections:
- net +15V: now also +12V.1, +12V.2, DOG2.1
- net GND: now also DOG2.2
Routing:
- net +15V: track 112.0 -> 177.1 mm
- net N$3: track 84.4 -> 78.0 mm
- net SW_RAW: track 24.2 -> 20.3 mm
- net N$22: track 15.5 -> 12.9 mm
- net N$29: track 15.2 -> 12.7 mm
- net N$28: track 14.7 -> 12.2 mm
- net V+WAS: track 103.7 -> 102.6 mm
- net N$23: track 15.1 -> 16.1 mm
- net N$34: track 14.8 -> 14.3 mm
Other:
- board text added: "+"
- board text added: "+12v"
- board text added: "+v O Com"
- board text removed: "+12 O C"
